Commit message: Updating to include adapter and simplify the collision objects.

File: robotiq_hande_description/urdf/grasp_push_frames.xacro (robot description, xacro)
@@ -3,25 +3,25 @@
   <xacro:macro name="grasp_push_frames" params="
     name:=''
-    prefix:=''
+    tf_prefix:=''
     marker_opacity:=0.5
     grasp_distance:=0.130
     finger_length:=0.046
     push_marker_size:=0.01">
-    <link name="${prefix}grasp_frame">
+    <link name="${tf_prefix}grasp_frame">
       <visual>
         <geometry>
           <sphere radius="0.007"/>
         </geometry>
-        <material name="${prefix}_green">
+        <material name="${tf_prefix}_green">
           <color rgba="0 1.0 0 ${marker_opacity}"/>
         </material>
       </visual>
     </link>
-    <joint name="${prefix}grasp_frame_joint" type="fixed">
-      <parent link="${prefix}gripper_base_link"/>
-      <child link="${prefix}grasp_frame"/>
+    <joint name="${tf_prefix}grasp_frame_joint" type="fixed">
+      <parent link="${tf_prefix}gripper_base_link"/>
+      <child link="${tf_prefix}grasp_frame"/>
       <origin xyz="0.0 0.0 ${grasp_distance}" rpy="0 0 0"/>
     </joint>
-    <link name="${prefix}push_frame_1">
+    <link name="${tf_prefix}push_frame_1">
       <visual>
         <origin xyz="0.0 0.0 ${push_marker_size / 8}" rpy="0 0 0"/>
@@ -29,15 +29,15 @@
           <box size="${push_marker_size} ${push_marker_size} ${push_marker_size / 4}"/>
         </geometry>
-        <material name="${prefix}_red">
+        <material name="${tf_prefix}_red">
           <color rgba="1.0 0 0 ${marker_opacity}"/>
         </material>
       </visual>
     </link>
-    <joint name="${prefix}push_frame_1_joint" type="fixed">
-      <parent link="${prefix}finger_1_link"/>
-      <child link="${prefix}push_frame_1"/>
+    <joint name="${tf_prefix}push_frame_1_joint" type="fixed">
+      <parent link="${tf_prefix}finger_1_link"/>
+      <child link="${tf_prefix}push_frame_1"/>
       <origin xyz="0.03 0.0 ${finger_length}" rpy="0 0 0"/>
     </joint>
-    <link name="${prefix}push_frame_2">
+    <link name="${tf_prefix}push_frame_2">
       <visual>
         <origin xyz="0.0 0.0 ${push_marker_size / 8} " rpy="0 0 0"/>
@@ -45,12 +45,12 @@
           <box size="${push_marker_size} ${push_marker_size} ${push_marker_size / 4} "/>
         </geometry>
-        <material name="${prefix}_red">
+        <material name="${tf_prefix}_red">
           <color rgba="1.0 0 0 ${marker_opacity}"/>
         </material>
       </visual>
     </link>
-    <joint name="${prefix}push_frame_2_joint" type="fixed">
-      <parent link="${prefix}finger_2_link"/>
-      <child link="${prefix}push_frame_2"/>
+    <joint name="${tf_prefix}push_frame_2_joint" type="fixed">
+      <parent link="${tf_prefix}finger_2_link"/>
+      <child link="${tf_prefix}push_frame_2"/>
       <origin xyz="0.03 0.0 ${finger_length}" rpy="0 0 0"/>
     </joint>

File: robotiq_hande_description/urdf/hande_fingers.xacro (robot description, xacro)
@@ -3,5 +3,5 @@
   <xacro:macro name="hande_fingers" params="
     name:=''
-    prefix:=''
+    tf_prefix:=''
     mount_x:=0.025
     mount_y:=0.0
@@ -11,5 +11,5 @@
     mount_yaw:=0.0
     scale:=0.001">
-    <link name="${prefix}finger_1_link">
+    <link name="${tf_prefix}finger_1_link">
       <inertial>
         <origin rpy="0 0 0" xyz="-0.02262 0.00759 0.00738"/>
@@ -20,17 +20,17 @@
           <origin xyz="0.0 0.0 0.0" rpy="0 0 0"/>
           <geometry>
-            <mesh filename="package://robotiq_hande_description/meshes/finger_1.stl" scale="${scale} ${scale} ${scale}"/>
+            <mesh filename="package://robotiq_hande_description/meshes/visual/finger_1.stl" scale="${scale} ${scale} ${scale}"/>
           </geometry>
-          <material name="${prefix}dark_gray"/>
+          <material name="${tf_prefix}dark_gray"/>
       </visual>
       <collision>
           <origin xyz="0.0 0.0 0.0" rpy="0 0 0"/>
           <geometry>
-            <mesh filename="package://robotiq_hande_description/meshes/finger_1.stl" scale="${scale} ${scale} ${scale}"/>
+            <mesh filename="package://robotiq_hande_description/meshes/collision/finger_1.stl" scale="${scale} ${scale} ${scale}"/>
           </geometry>
-          <material name="${prefix}dark_gray"/>
+          <material name="${tf_prefix}dark_gray"/>
       </collision>
     </link>
-    <link name="${prefix}finger_2_link">
+    <link name="${tf_prefix}finger_2_link">
       <inertial>
         <origin rpy="0 0 0" xyz="0.02262 -0.00759 0.00738"/>
@@ -41,30 +41,30 @@
           <origin xyz="0.0 0.0 0.0" rpy="0 0 0"/>
           <geometry>
-            <mesh filename="package://robotiq_hande_description/meshes/finger_1.stl" scale="${scale} ${scale} ${scale}"/>
+            <mesh filename="package://robotiq_hande_description/meshes/visual/finger_1.stl" scale="${scale} ${scale} ${scale}"/>
           </geometry>
-          <material name="${prefix}dark_gray"/>
+          <material name="${tf_prefix}dark_gray"/>
       </visual>
       <collision>
           <origin xyz="0.0 0.0 0.0" rpy="0 0 0"/>
           <geometry>
-            <mesh filename="package://robotiq_hande_description/meshes/finger_1.stl" scale="${scale} ${scale} ${scale}"/>
+            <mesh filename="package://robotiq_hande_description/meshes/collision/finger_1.stl" scale="${scale} ${scale} ${scale}"/>
           </geometry>
-          <material name="${prefix}dark_gray"/>
+          <material name="${tf_prefix}dark_gray"/>
       </collision>
     </link>
-    <joint name="${prefix}finger_1_joint" type="prismatic">
+    <joint name="${tf_prefix}finger_1_joint" type="prismatic">
       <origin rpy="${mount_roll} ${mount_pitch} ${mount_yaw + pi}" xyz="${mount_x} ${mount_y} ${mount_z}"/>
-      <parent link="${prefix}gripper_base_link"/>
-      <child link="${prefix}finger_1_link"/>
+      <parent link="${tf_prefix}gripper_base_link"/>
+      <child link="${tf_prefix}finger_1_link"/>
       <axis xyz="1 0 0"/>
       <limit effort="130" lower="0" upper="0.025" velocity="0.15"/>
     </joint>
-    <joint name="${prefix}finger_2_joint" type="prismatic">
+    <joint name="${tf_prefix}finger_2_joint" type="prismatic">
       <origin rpy="${mount_roll} ${mount_pitch} ${mount_yaw}" xyz="${-mount_x} ${-mount_y} ${mount_z}"/>
-      <parent link="${prefix}gripper_base_link"/>
-      <child link="${prefix}finger_2_link"/>
+      <parent link="${tf_prefix}gripper_base_link"/>
+      <child link="${tf_prefix}finger_2_link"/>
       <axis xyz="1 0 0"/>
       <limit effort="130" lower="0" upper="0.025" velocity="0.15"/>
-      <mimic joint="${prefix}finger_1_joint" multiplier="1" offset="0"/>
+      <mimic joint="${tf_prefix}finger_1_joint" multiplier="1" offset="0"/>
     </joint>
   </xacro:macro>

File: robotiq_hande_description/urdf/robotiq_gripper_hande.urdf.xacro (robot description, xacro)
@@ -2,5 +2,5 @@
 <robot xmlns:xacro="http://wiki.ros.org/xacro" name="robotiq_hande">
   <xacro:arg name="name" default="RobotiqGripperHandeHardwareInterface"/>
-  <xacro:arg name="prefix" default=""/>
+  <xacro:arg name="tf_prefix" default=""/>
   <xacro:arg name="use_fake_hardware" default="false"/>
   <xacro:arg name="com_port" default="/dev/ttyACM0"/>
@@ -9,8 +9,8 @@
   <xacro:include filename="$(find robotiq_hande_description)/urdf/grasp_push_frames.xacro"/>
   <link name="world"/>
-  <xacro:robotiq_hande name="$(arg name)" prefix="$(arg prefix)" parent="world" use_fake_hardware="$(arg use_fake_hardware)" com_port="$(arg com_port)">
+  <xacro:robotiq_hande name="$(arg name)" tf_prefix="$(arg tf_prefix)" parent="world" use_fake_hardware="$(arg use_fake_hardware)" com_port="$(arg com_port)">
     <origin xyz="0 0 0" rpy="0 0 0"/>
   </xacro:robotiq_hande>
-  <xacro:hande_fingers name="$(arg name)" prefix="$(arg prefix)"/>
-  <xacro:grasp_push_frames name="$(arg name)" prefix="$(arg prefix)"/>
+  <xacro:hande_fingers name="$(arg name)" tf_prefix="$(arg tf_prefix)"/>
+  <xacro:grasp_push_frames name="$(arg name)" tf_prefix="$(arg tf_prefix)"/>
 </robot>

File: robotiq_hande_description/urdf/robotiq_hande.ros2_control.xacro (robot description, xacro)
@@ -3,5 +3,5 @@
   <xacro:macro name="robotiq_hande_ros2_control" params="
       name:=robotiq
-      prefix
+      tf_prefix
       use_fake_hardware:=true
       fake_sensor_commands:=false
@@ -20,5 +20,5 @@
         </xacro:unless>
       </hardware>
-      <joint name="${prefix}finger_1_joint">
+      <joint name="${tf_prefix}finger_1_joint">
         <param name="initial_position">0.00</param>
         <command_interface name="position"/>

File: robotiq_hande_description/urdf/robotiq_hande.xacro (robot description, xacro)
@@ -5,5 +5,5 @@
   <xacro:macro name="robotiq_hande" params="
     name
-    prefix
+    tf_prefix
     parent
     *origin
@@ -11,8 +11,8 @@
     fake_sensor_commands:=false
     com_port:=/dev/ttyUSB1">
-    <material name="${prefix}dark_gray">
+    <material name="${tf_prefix}dark_gray">
       <color rgba="0.2 0.2 0.2 1"/>
     </material>
-    <material name="${prefix}black">
+    <material name="${tf_prefix}black">
       <color rgba="0 0 0 1"/>
     </material>
@@ -20,15 +20,36 @@
     <xacro:robotiq_hande_ros2_control
         name="${name}"
-        prefix="${prefix}"
+        tf_prefix="${tf_prefix}"
         use_fake_hardware="${use_fake_hardware}"
         fake_sensor_commands="${fake_sensor_commands}"
         com_port="${com_port}"
         />
-    <joint name="${prefix}gripper_base_joint" type="fixed">
+    <joint name="${tf_prefix}gripper_adapter_joint" type="fixed">
       <parent link="${parent}"/>
-      <child link="${prefix}gripper_base_link"/>
+      <child link="${tf_prefix}robotiq_hande_cb_adapter"/>
       <xacro:insert_block name="origin"/>
     </joint>
-    <link name="${prefix}gripper_base_link">
+    <link name="${tf_prefix}robotiq_hande_cb_adapter">
+      <origin xyz="0 0 0" rpy="0 0 0" />
+      <visual>
+        <geometry>
+          <mesh filename="package://robotiq_hande_description/meshes/visual/robotiq_hande_cb_adapter.dae"/>
+        </geometry>
+        <material name="${tf_prefix}black"/>
+      </visual>
+      <collision>
+        <origin xyz="0 0 0.006" rpy="0 0 0" />
+        <geometry>
+          <cylinder length="0.018" radius="0.038"/>
+        </geometry>
+        <material name="${tf_prefix}black"/>
+      </collision>
+    </link>
+    <joint name="${tf_prefix}gripper_base_joint" type="fixed">
+      <parent link="${tf_prefix}robotiq_hande_cb_adapter"/>
+      <child link="${tf_prefix}gripper_base_link"/>
+      <origin xyz="0.0 0.0 0.011" rpy="0 0 0"/>
+    </joint>
+    <link name="${tf_prefix}gripper_base_link">
       <inertial>
         <origin xyz="0 0 0.04607" rpy="0 0 0" />
@@ -39,27 +60,27 @@
         <origin xyz="0 0 0" rpy="0 0 0" />
         <geometry>
-          <mesh filename="package://robotiq_hande_description/meshes/hand-e.dae" scale="0.001 0.001 0.001"/>
+          <mesh filename="package://robotiq_hande_description/meshes/visual/hande.dae" scale="0.001 0.001 0.001"/>
         </geometry>
-        <material name="${prefix}black"/>
+        <material name="${tf_prefix}black"/>
       </visual>
       <collision>
-        <origin xyz="0 0 0" rpy="0 0 0" />
+        <origin xyz="0 0 0.050" rpy="0 0 0" />
         <geometry>
-          <mesh filename="package://robotiq_hande_description/meshes/hand-e.dae" scale="0.001 0.001 0.001"/>
+          <cylinder length="0.10" radius="0.038"/>
         </geometry>
-        <material name="${prefix}black"/>
+        <material name="${tf_prefix}black"/>
       </collision>
     </link>
-    <joint name="${prefix}gripper_palm_joint" type="fixed">
-      <parent link="${prefix}gripper_base_link"/>
-      <child link="${prefix}gripper_palm_link"/>
+    <joint name="${tf_prefix}gripper_palm_joint" type="fixed">
+      <parent link="${tf_prefix}gripper_base_link"/>
+      <child link="${tf_prefix}gripper_palm_link"/>
       <origin xyz="0.0 0.0 0.0988" rpy="0 0 0"/>
     </joint>
-    <link name="${prefix}gripper_palm_link">
-    <visual>
+    <link name="${tf_prefix}gripper_palm_link">
+      <visual>
         <geometry>
           <sphere radius="0.007"/>
         </geometry>
-        <material name="${prefix}_green">
+        <material name="${tf_prefix}_green">
           <color rgba="0 1.0 0 0.5"/>
         </material>
