Commit message: Support gz in ros2 control config

File: robotiq_hande_description/urdf/robotiq_hande.ros2_control.xacro (robot description, xacro)
@@ -4,4 +4,5 @@
       name:=robotiq
       tf_prefix
+      sim_ignition:=false
       use_fake_hardware:=true
       fake_sensor_commands:=false
@@ -12,5 +13,8 @@
           <plugin>fake_components/GenericSystem</plugin>
         </xacro:if>
-        <xacro:unless value="${use_fake_hardware}">
+        <xacro:if value="${sim_ignition}">
+            <plugin>ign_ros2_control/IgnitionSystem</plugin>
+        </xacro:if>
+        <xacro:unless value="${use_fake_hardware or sim_ignition}">
             <plugin>robotiq_driver_hande/RobotiqGripperHandeHardwareInterface</plugin>
             <param name="gripper_closed_position">0.059</param>
@@ -21,11 +25,16 @@
       </hardware>
       <joint name="${tf_prefix}finger_1_joint">
-        <param name="initial_position">0.00</param>
         <command_interface name="position"/>
         <state_interface name="position">
-          <param name="initial_value">0.0</param>
+          <param name="initial_value">0.020</param>
         </state_interface>
         <state_interface name="velocity"/>
       </joint>
+      <xacro:if value="${use_fake_hardware or sim_ignition}">
+        <joint name="${tf_prefix}finger_2_joint">
+          <param name="mimic">${tf_prefix}finger_1_joint</param>
+          <param name="multiplier">1</param>
+        </joint>
+      </xacro:if>
       <!-- Only add this with fake hardware mode -->
       <xacro:if value="${use_fake_hardware}">

File: robotiq_hande_description/urdf/robotiq_hande.xacro (robot description, xacro)
@@ -25,4 +25,5 @@
         name="${name}"
         tf_prefix="${tf_prefix}"
+        sim_ignition="${sim_ignition}"
         use_fake_hardware="${use_fake_hardware}"
         fake_sensor_commands="${fake_sensor_commands}"
