Commit message: Adding a palm frame for calibration.

File: robotiq_hande_description/urdf/robotiq_hande.xacro (robot description, xacro)
@@ -51,4 +51,19 @@
       </collision>
     </link>
+    <joint name="${prefix}gripper_palm_joint" type="fixed">
+      <parent link="${parent}"/>
+      <child link="${prefix}gripper_palm_link"/>
+      <origin xyz="0.0 0.0 0.0988" rpy="0 0 0"/>
+    </joint>
+    <link name="${prefix}gripper_palm_link">
+    <visual>
+        <geometry>
+          <sphere radius="0.007"/>
+        </geometry>
+        <material name="${prefix}_green">
+          <color rgba="0 1.0 0 0.5"/>
+        </material>
+      </visual>
+    </link>
   </xacro:macro>
 </robot>

Commit message: Fixing a bug for the palm frame.

File: robotiq_hande_description/urdf/robotiq_hande.xacro (robot description, xacro)
@@ -52,5 +52,5 @@
     </link>
     <joint name="${prefix}gripper_palm_joint" type="fixed">
-      <parent link="${parent}"/>
+      <parent link="${prefix}gripper_base_link"/>
       <child link="${prefix}gripper_palm_link"/>
       <origin xyz="0.0 0.0 0.0988" rpy="0 0 0"/>

Commit message: Adding inertia TODO.

File: robotiq_hande_description/urdf/robotiq_hande.xacro (robot description, xacro)
@@ -31,4 +31,10 @@
     </joint>
     <link name="${tf_prefix}robotiq_hande_cb_adapter">
+      <!--TODO set proper inertia-->
+      <inertial>
+        <origin rpy="0 0 0" xyz="0.0 0.0 0.0"/>
+        <mass value="0.0"/>
+        <inertia ixx="0.0" ixy="0.0" ixz="0.0" iyy="0.0" iyz="0.0" izz="0.0"/>
+      </inertial>
       <origin xyz="0 0 0" rpy="0 0 0" />
       <visual>

Commit message: Add path modifications for mesh files to support gazebo path requirements at launch

File: robotiq_hande_description/urdf/robotiq_hande.xacro (robot description, xacro)
@@ -3,4 +3,5 @@
   <xacro:arg name="use_fake_hardware" default="false"/>
   <xacro:include filename="$(find robotiq_hande_description)/urdf/robotiq_hande.ros2_control.xacro"/>
+  <xacro:include filename="$(find robotiq_hande_description)/urdf/gen_mesh.xacro"/>
   <xacro:macro name="robotiq_hande" params="
     name
@@ -8,4 +9,5 @@
     parent
     *origin
+    sim_ignition:=false
     use_fake_hardware:=false
     fake_sensor_commands:=false
@@ -17,4 +19,6 @@
       <color rgba="0 0 0 1"/>
     </material>
+    <!-- if ignition or gazebo - need to use absolute paths instead of relative, applies locally -->
+    <xacro:property name="force_abs_paths" value="$(arg sim_ignition)" />
     <!-- ros2 control instance -->
     <xacro:robotiq_hande_ros2_control
@@ -40,5 +44,8 @@
       <visual>
         <geometry>
-          <mesh filename="package://robotiq_hande_description/meshes/visual/robotiq_hande_cb_adapter.dae"/>
+          <xacro:gen_mesh
+            force_abs_path="${force_abs_paths}"
+            pkg_name="robotiq_hande_description"
+            file_path="meshes/visual/robotiq_hande_cb_adapter.dae" />
         </geometry>
         <material name="${tf_prefix}black"/>
@@ -66,5 +73,9 @@
         <origin xyz="0 0 0" rpy="0 0 0" />
         <geometry>
-          <mesh filename="package://robotiq_hande_description/meshes/visual/hande.dae" scale="0.001 0.001 0.001"/>
+          <xacro:gen_mesh
+            force_abs_path="${force_abs_paths}"
+            pkg_name="robotiq_hande_description"
+            file_path="meshes/visual/hande.dae"
+            scale="0.001 0.001 0.001"/>
         </geometry>
         <material name="${tf_prefix}black"/>

Commit message: adding mass properties for adapter

File: robotiq_hande_description/urdf/robotiq_hande.xacro (robot description, xacro)
@@ -38,9 +38,9 @@
     </joint>
     <link name="${tf_prefix}robotiq_hande_cb_adapter">
-      <!--TODO set proper inertia-->
+      <!--Not sure if these are right, based on the robotiq numbers for ur_to_robotiq_link-->
       <inertial>
-        <origin rpy="0 0 0" xyz="0.0 0.0 0.0"/>
-        <mass value="0.0"/>
-        <inertia ixx="0.0" ixy="0.0" ixz="0.0" iyy="0.0" iyz="0.0" izz="0.0"/>
+        <mass value="0.01" />
+        <origin xyz="0 0 0" />
+        <inertia ixx="0.000044" ixy="0.0" ixz="0.0" iyy="0.000027" iyz="0.0" izz="0.000027" />
       </inertial>
       <origin xyz="0 0 0" rpy="0 0 0" />

Commit message: updating the sim ignition to reference the macro param, not global arg

File: robotiq_hande_description/urdf/robotiq_hande.xacro (robot description, xacro)
@@ -20,5 +20,5 @@
     </material>
     <!-- if ignition or gazebo - need to use absolute paths instead of relative, applies locally -->
-    <xacro:property name="force_abs_paths" value="$(arg sim_ignition)" />
+    <xacro:property name="force_abs_paths" value="${sim_ignition}" />
     <!-- ros2 control instance -->
     <xacro:robotiq_hande_ros2_control

Commit message: removing unnecessary green sphere on palm link

File: robotiq_hande_description/urdf/robotiq_hande.xacro (robot description, xacro)
@@ -97,14 +97,5 @@
       <origin xyz="0.0 0.0 0.0988" rpy="0 0 0"/>
     </joint>
-    <link name="${tf_prefix}gripper_palm_link">
-      <visual>
-        <geometry>
-          <sphere radius="0.007"/>
-        </geometry>
-        <material name="${tf_prefix}_green">
-          <color rgba="0 1.0 0 0.5"/>
-        </material>
-      </visual>
-    </link>
+    <link name="${tf_prefix}gripper_palm_link"/>
   </xacro:macro>
 </robot>
