Commit message: updated masses for the hande

File: robotiq_hande_description/urdf/robotiq_hande.xacro (robot description, xacro)
@@ -39,6 +39,7 @@
     <link name="${tf_prefix}robotiq_hande_cb_adapter">
       <!--Not sure if these are right, based on the robotiq numbers for ur_to_robotiq_link-->
+      <!-- Mass is a temporary value. Measured: ur_realsense_mount + robotiq_hande_adapter = 269.5 g -->
       <inertial>
-        <mass value="0.01" />
+        <mass value="0.1695" />
         <origin xyz="0 0 0" />
         <inertia ixx="0.000044" ixy="0.0" ixz="0.0" iyy="0.000027" iyz="0.0" izz="0.000027" />
@@ -68,7 +69,8 @@
     </joint>
     <link name="${tf_prefix}gripper_base_link">
+      <!-- Updated mass including finger attachment points -->
       <inertial>
         <origin xyz="0 0 0.04607" rpy="0 0 0" />
-        <mass value="0.86387" />
+        <mass value="0.901" />
         <inertia ixx="1017560E-9" ixy="0" ixz="2235E-9" iyy="1028041E-9" iyz="0" izz="489810E-9" />
       </inertial>

Commit message: update inertia and mass properties

File: robotiq_hande_description/urdf/robotiq_hande.xacro (robot description, xacro)
@@ -39,9 +39,9 @@
     <link name="${tf_prefix}robotiq_hande_cb_adapter">
       <!--Not sure if these are right, based on the robotiq numbers for ur_to_robotiq_link-->
-      <!-- Mass is a temporary value. Measured: ur_realsense_mount + robotiq_hande_adapter = 269.5 g -->
+      <!-- Mass is estimated. Combined mass of ur_realsense_mount and robotiq_hande_adapter is 269.5 g -->
       <inertial>
-        <mass value="0.1695" />
-        <origin xyz="0 0 0" />
-        <inertia ixx="0.000044" ixy="0.0" ixz="0.0" iyy="0.000027" iyz="0.0" izz="0.000027" />
+        <mass value="0.2174" />
+        <origin xyz="-1.9561273e-04  1.6716577e-03  5.1888253e-03" />
+        <inertia ixx="4.1495874e-05" ixy="-3.5226788e-08" ixz="6.5573497e-09" iyy="5.2040925e-05" iyz="4.7369283e-07" izz="9.0288619e-05" />
       </inertial>
       <origin xyz="0 0 0" rpy="0 0 0" />
@@ -71,7 +71,7 @@
       <!-- Updated mass including finger attachment points -->
       <inertial>
-        <origin xyz="0 0 0.04607" rpy="0 0 0" />
+        <origin xyz="0 0 4.8470158e-02" rpy="0 0 0" />
         <mass value="0.901" />
-        <inertia ixx="1017560E-9" ixy="0" ixz="2235E-9" iyy="1028041E-9" iyz="0" izz="489810E-9" />
+        <inertia ixx="1.1281390e-03" ixy="0" ixz="0" iyy="1.1556521e-03" iyz="0" izz="5.3230056e-04" />
       </inertial>
       <visual>
