Commit message: increase force limit to match datasheet

File: robotiq_hande_description/urdf/hande_fingers.xacro (robot description, xacro)
@@ -58,5 +58,5 @@
       <child link="${tf_prefix}finger_1_link"/>
       <axis xyz="1 0 0"/>
-      <limit effort="130" lower="0" upper="0.025" velocity="0.15"/>
+      <limit effort="185" lower="0" upper="0.025" velocity="0.15"/>
     </joint>
     <joint name="${tf_prefix}finger_2_joint" type="prismatic">
@@ -65,5 +65,5 @@
       <child link="${tf_prefix}finger_2_link"/>
       <axis xyz="1 0 0"/>
-      <limit effort="130" lower="0" upper="0.025" velocity="0.15"/>
+      <limit effort="185" lower="0" upper="0.025" velocity="0.15"/>
       <mimic joint="${tf_prefix}finger_1_joint" multiplier="1" offset="0"/>
     </joint>
